File: BuoyPower.kicad_pcb (KiCad board)
At the start: 2 copper layers, 65 x 30 mm, 33 parts, among them J1 Pololu-3782, J2 Conn_01x02_Male, J4 Conn_01x02_Male, J9 Screw_Terminal_01x04, U10 74LVC2G02, U11 SN74AUP1G32, U3 INA219AxD, U8 DS3231M, U9 74LVC1GU04

Commit message: PiShield!!
Parts:
- removed C14: .1uf, Capacitor_SMD:C_0805_2012Metric_Pad1.18x1.45mm_HandSolder
- removed H4: MountingHole, MountingHole:MountingHole_3.2mm_M3_Pad_Via
- removed J9: Screw_Terminal_01x04, TerminalBlock_4Ucon:TerminalBlock_4Ucon_1x04_P3.50mm_Horizontal
- removed JP1: SolderJumper_3_Bridged12, Jumper:SolderJumper-3_P1.3mm_Bridged12_Pad1.0x1.5mm
- removed JP26: SolderJumper_2_Open, Connector_PinHeader_2.54mm:PinHeader_1x02_P2.54mm_Vertical
- removed JP41: SolderJumper_2_Bridged, Jumper:SolderJumper-2_P1.3mm_Bridged_Pad1.0x1.5mm
- removed U10: 74LVC2G02, SOP65P400X110-8N:SOP65P400X110-8N
- added C2: 10uF, Capacitor_SMD:C_0805_2012Metric_Pad1.18x1.45mm_HandSolder, F.Cu at (141.4, 114.3)
- added H5: MountingHole, MountingHole:MountingHole_2.2mm_M2, F.Cu at (168.5, 98.4)
- added J10: Conn_02x20_Odd_Even, Connector_PinSocket_2.54mm:PinSocket_2x20_P2.54mm_Vertical, B.Cu at (176.2, 74.0)
- added J5: Conn_01x03, Connector_JST:JST_XH_S3B-XH-A_1x03_P2.50mm_Horizontal, F.Cu at (152.4, 75.3)
- added J6: Conn_01x04, Connector_JST:JST_SH_SM04B-SRSS-TB_1x04-1MP_P1.00mm_Horizontal, F.Cu at (138.2, 69.5)
- added J7: Conn_01x02_Male, Connector_JST:JST_XH_S2B-XH-A_1x02_P2.50mm_Horizontal, F.Cu at (134.9, 77.5)
- added J8: Conn_01x04, Connector_JST:JST_XH_S4B-XH-A_1x04_P2.50mm_Horizontal, F.Cu at (167.3, 75.3)
- added JP3: SolderJumper_2_Open, Jumper:SolderJumper-2_P1.3mm_Open_Pad1.0x1.5mm, F.Cu at (148.3, 124.8)
- added R1: 120k, Resistor_SMD:R_0805_2012Metric_Pad1.20x1.40mm_HandSolder, F.Cu at (141.4, 118.4)
- added S1: EG1213, EG1213:SW_EG1213, F.Cu at (132.6, 114.6)
- BT2: moved to B.Cu
- H1: footprint MountingHole:MountingHole_3.2mm_M3_Pad_Via -> MountingHole:MountingHole_2.2mm_M2
- H2, H3: footprint MountingHole:MountingHole_3.2mm_M3_Pad_Via -> MountingHole:MountingHole_3.2mm_M3
- J1: footprint Connector_PinHeader_2.54mm:PinHeader_1x05_P2.54mm_Vertical -> ADAFRUIT_QT_PY:Pololu-3782
- J2: value Conn_01x02_Male -> Conn_01x05; footprint TerminalBlock_4Ucon:TerminalBlock_4Ucon_1x02_P3.50mm_Horizontal -> Connector_PinHeader_2.54mm:PinHeader_1x05_P2.54mm_Vertical
- J4: footprint TerminalBlock_4Ucon:TerminalBlock_4Ucon_1x02_P3.50mm_Horizontal -> Connector_JST:JST_XH_S2B-XH-A_1x02_P2.50mm_Horizontal
- JP2: value SolderJumper_3_Bridged12 -> SolderJumper_2_Open; footprint Jumper:SolderJumper-3_P1.3mm_Bridged12_Pad1.0x1.5mm -> Jumper:SolderJumper-2_P1.3mm_Open_Pad1.0x1.5mm
- JP4: value SolderJumper_3_Open -> SolderJumper_2_Open; footprint Connector_PinHeader_2.54mm:PinHeader_1x03_P2.54mm_Vertical -> Jumper:SolderJumper-2_P1.3mm_Open_Pad1.0x1.5mm
- moved H2 88.5 mm to (128.5, 69.2), turned to 180 degrees
- moved BT2 84.8 mm to (151.9, 120.7), turned to 0 degrees
- moved J4 82.3 mm to (134.9, 87.7), turned to -90 degrees
- moved H1 70.4 mm to (152.5, 85.0)
- moved C15 70.1 mm to (143.0, 125.7), turned to 180 degrees
- moved J2 67.2 mm to (127.5, 106.0), turned to 180 degrees
- moved JP4 65.9 mm to (148.3, 122.3)
- moved U11 65.4 mm to (143.3, 122.7), turned to 180 degrees
- moved R15 63.5 mm to (145.2, 113.2), turned to -90 degrees
- moved C13 63.3 mm to (148.2, 117.6)
- moved U9 63.3 mm to (145.2, 117.6)
- moved JP2 60.5 mm to (138.7, 116.6), turned to 90 degrees
- moved JP42 59.4 mm to (149.1, 113.1)
- moved J1 56.7 mm to (169.4, 84.1), turned to -90 degrees
- moved U8 56.5 mm to (160.7, 114.3), turned to 0 degrees
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Connections:
- BT2 pad 1: +BATT -> Vbat
- C13 pad 2: +BATT -> Vbat
- C15 pad 2: +BATT -> Vbat
- J1 pad 1: /REG_EN -> +5V
- J1 pad 2: /PowerMonitor/VOUT -> GND
- J1 pad 3: GND1 -> GND
- J1 pad 4: GND1 -> /PowerMonitor/VOUT
- J1 pad 5: +5V -> /REG_EN
- J2 pad 1: GND -> /HOLD
- J2 pad 2: VBUS -> /SCL
- J4 pad 2: +BATT -> BATT_IN
- JP2 pad 1: /PowerTimer/AOUT -> Net-(JP2-A)
- JP2 pad 2: Net-(U11-Pad1) -> Net-(JP2-B)
- JP4 pad 1: Net-(U11-Pad4) -> /PowerTimer/NINT
- JP4 pad 2: /REG_EN -> Net-(JP4-B)
- R10 pad 1: +BATT -> BATT_IN
- R11 pad 1: +BATT -> BATT_IN
- R13 pad 1: /PowerTimer/SCL -> /SCL
- R14 pad 1: /PowerTimer/SDA -> /SDA
- R15 pad 1: +BATT -> Vbat
- U11 pad 1: Net-(U11-Pad1) -> Net-(JP3-B)
- U11 pad 2: /PowerTimer/POWER_HOLD -> Net-(JP4-B)
- U11 pad 4: Net-(U11-Pad4) -> Net-(JP2-A)
- U11 pad 5: +BATT -> Vbat
- U3 pad 1: /PowerMonitor/A1 -> GND
- U3 pad 2: /PowerMonitor/A0 -> GND
- U3 pad 3: /PowerMonitor/SDA -> /SDA
- U3 pad 4: /PowerMonitor/SCL -> /SCL
- U8 pad 1: Net-(JP41-A) -> unconnected-(U8-32KHZ)
- U8 pad 14: +BATT -> Vbat
- U8 pad 15: /PowerTimer/SDA -> /SDA
- U8 pad 16: /PowerTimer/SCL -> /SCL
- U9 pad 5: +BATT -> Vbat
Routing:
- net /SDA: track 0.00 -> 140.5 mm, vias 0 -> 9
- net /SCL: track 0.00 -> 132.9 mm, vias 0 -> 7
- net VBUS: track 0.00 -> 128.4 mm, vias 0 -> 3
- net /HOLD: track 0.00 -> 100.0 mm, vias 0 -> 1
- net GND: track 0.00 -> 75.1 mm, vias 0 -> 45
- net BATT_IN: track 0.00 -> 68.5 mm
- net Vbat: track 0.00 -> 65.9 mm, vias 0 -> 2
- net /REG_EN: track 0.00 -> 47.2 mm, vias 0 -> 2
- net +5V: track 0.00 -> 27.4 mm
- net /PowerMonitor/VOUT: track 0.00 -> 26.6 mm
- net Net-(JP2-B): track 0.00 -> 12.2 mm, vias 0 -> 1
- net Net-(JP42-A): track 0.00 -> 7.53 mm
- net /PowerTimer/NINT: track 0.00 -> 7.50 mm
- net Net-(JP2-A): track 0.00 -> 6.92 mm
- net /PowerTimer/INT: track 0.00 -> 6.68 mm
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- added copper zone on B.Cu, net GND
- added copper zone on F.Cu, net GND
Other:
- board size 65 x 30 mm -> 56 x 65.5 mm

Commit message: Ready to order.
Parts:
- added D1: BAT20J, Diode_SMD:D_SOD-323_HandSoldering, F.Cu at (134.7, 103.6)
- added D2: BAT20J, Diode_SMD:D_SOD-323_HandSoldering, F.Cu at (138.4, 103.6)
- added J9: Conn_01x02_Male, Connector_PinHeader_2.54mm:PinHeader_1x02_P2.54mm_Vertical, F.Cu at (164.3, 128.5)
- added JP1: SolderJumper_2_Bridged, Jumper:SolderJumper-2_P1.3mm_Bridged_Pad1.0x1.5mm, F.Cu at (136.7, 107.7)
- R15: value 10k -> 470k
- U11: value SN74AUP1G32 -> SN74AHC1G32
- U9: value 74LVC1GU04 -> 74AHC1GU04
- moved JP42 2.28 mm to (150.9, 114.6), turned to 180 degrees
- moved JP2 0.51 mm to (138.2, 116.6)
- turned S1 to -90 degrees
Connections:
- BT2 pad 1: Vbat -> Net-(J9-Pin_2)
- C13 pad 2: Vbat -> VCC
- C15 pad 2: Vbat -> VCC
- R15 pad 1: Vbat -> VCC
- S1 pad 1: Vbat -> VCC
- U11 pad 5: Vbat -> VCC
- U8 pad 14: Vbat -> Net-(J9-Pin_2)
- U9 pad 5: Vbat -> VCC
Routing:
- net Vbat: track 65.9 -> 0.00 mm, vias 2 -> 0
- net VCC: track 0.00 -> 64.9 mm, vias 0 -> 2
- net Net-(J9-Pin_2): track 0.00 -> 45.8 mm, vias 0 -> 2
- net GND: track 75.1 -> 90.8 mm
- net /HOLD: track 100.0 -> 114.5 mm
- net Net-(D1-K): track 0.00 -> 5.91 mm
- net VBUS: track 128.4 -> 132.2 mm, vias 3 -> 4
- net Net-(JP42-A): track 7.53 -> 5.40 mm
- net Net-(JP2-B): track 12.2 -> 11.1 mm, vias 1 -> 0
- net /PowerTimer/INT: track 6.68 -> 7.31 mm
- net /REG_EN: track 47.2 -> 47.6 mm, vias 2 -> 4
Other:
- board text added: "AUTO"
- board text added: "CR2032+"
- board text added: "GND"
- board text added: "ON"

Commit message: Pushing to github
Parts:
- H2, H3: footprint MountingHole:MountingHole_3.2mm_M3 -> MountingHole:MountingHole_3.2mm_M3_Pad_Via
- moved J6 0.89 mm to (138.2, 68.6)
Other:
- board text added: "9/4/23"
- board text added: "DIY Aquanauts"
- board text added: "Power Controller"
