File: BuoyPower.kicad_pcb (KiCad board)
At the start: 2 copper layers, 56 x 65.5 mm, 40 parts, among them J1 Pololu-3782, J10 Conn_02x20_Odd_Even, J2 Conn_01x05, J4 Conn_01x02_Male, J5 Conn_01x03, J6 Conn_01x04, J7 Conn_01x02_Male, J8 Conn_01x04, J9 Conn_01x02_Male, U11 SN74AHC1G32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

Commit message: Post-build updates
Parts:
- removed C2: 10uF, Capacitor_SMD:C_0805_2012Metric_Pad1.18x1.45mm_HandSolder
- removed JP2: SolderJumper_2_Open, Jumper:SolderJumper-2_P1.3mm_Open_Pad1.0x1.5mm
- removed R1: 120k, Resistor_SMD:R_0805_2012Metric_Pad1.20x1.40mm_HandSolder
- added Q1: IRLML2502, Package_TO_SOT_SMD:SOT-23, F.Cu at (139.6, 114.8)
- C1: value 0.1uf -> 0.1uF
- C12, C13, C15: value .1uf -> 0.1uF
- C3: value 100n -> 0.1uF
- JP3, JP4: footprint Jumper:SolderJumper-2_P1.3mm_Open_Pad1.0x1.5mm -> Jumper:SolderJumper-2_P1.3mm_Bridged_Pad1.0x1.5mm
- moved JP3 0.13 mm to (148.3, 125.0)
- moved JP4 0.13 mm to (148.3, 122.4)
Connections:
- S1 pad 2: /REG_EN -> Net-(S1-Pad2)
- S1 pad 3: Net-(JP2-B) -> Net-(U11-Pad4)
- U11 pad 4: Net-(JP2-A) -> Net-(U11-Pad4)
Routing:
- net Net-(U11-Pad4): track 0.00 -> 11.5 mm
- net Net-(JP2-B): track 11.1 -> 0.00 mm
- net Net-(JP2-A): track 6.93 -> 0.00 mm
- net Net-(S1-Pad2): track 0.00 -> 6.53 mm
- net /REG_EN: track 47.6 -> 42.1 mm
- net BATT_IN: track 68.5 -> 67.3 mm

Commit message: technically ok
Parts:
- removed JP42: SolderJumper_2_Bridged, Jumper:SolderJumper-2_P1.3mm_Bridged_Pad1.0x1.5mm
- removed S1: EG1213, EG1213:SW_EG1213
- removed U11: SN74AHC1G32, Package_TO_SOT_SMD:SOT-23-5_HandSoldering
- added ?: , , F.Cu at (142.0, 88.9)
- added D3: LED, LED_SMD:LED_0805_2012Metric, F.Cu at (133.9, 121.3)
- added R1: 10k, Resistor_SMD:R_0805_2012Metric_Pad1.20x1.40mm_HandSolder, F.Cu at (133.9, 123.6)
- added SW1: SW_Push_DPDT, JS202011SCQN:SW_JS202011SCQN, F.Cu at (130.4, 115.2)
- added U1: 74AHC1G02, Package_TO_SOT_SMD:SOT-23-5_HandSoldering, F.Cu at (148.8, 117.3)
- moved R15 17.6 mm to (159.3, 123.7), turned to 180 degrees
- moved U9 11.4 mm to (154.8, 123.7), turned to 180 degrees
- moved C13 11.3 mm to (154.8, 126.7), turned to 180 degrees
- moved C1 9.27 mm to (149.1, 93.0)
- moved C3 9.27 mm to (143.0, 88.9)
- moved R10 9.27 mm to (143.0, 82.5)
- moved R11 9.27 mm to (140.0, 86.6)
- moved R12 9.27 mm to (146.1, 86.6)
- moved U3 9.27 mm to (144.3, 94.6)
- moved C15 9.08 mm to (145.8, 117.1), turned to 90 degrees
- moved JP3 3.21 mm to (146.6, 122.3), turned to 90 degrees
- moved Q1 1.40 mm to (139.7, 116.2), turned to 0 degrees
- moved JP4 0.77 mm to (149.1, 122.3), turned to 90 degrees
- moved J2 0.76 mm to (128.3, 106.0)
Connections:
- Q1 pad 1: Net-(S1-Pad2) -> /PowerTimer/EN_OUT
- U8 pad 3: Net-(JP42-A) -> /PowerTimer/INT
Routing:
- net VBUS: track 132.2 -> 47.5 mm, vias 4 -> 5
- net BATT_IN: track 67.3 -> 7.18 mm, vias 0 -> 5
- net VCC: track 64.9 -> 29.1 mm, vias 2 -> 7
- net /SDA: track 140.5 -> 124.8 mm, vias 9 -> 2
- net GND: track 90.6 -> 75.1 mm, vias 45 -> 28
- net /HOLD: track 114.5 -> 103.0 mm
- net Net-(U11-Pad4): track 11.5 -> 0.00 mm
- net /SCL: track 132.9 -> 122.9 mm, vias 7 -> 2
- net /PowerMonitor/VOUT: track 26.6 -> 36.2 mm
- net /PowerTimer/TEST_OUT: track 0.00 -> 9.48 mm
- net /PowerTimer/INT: track 7.31 -> 16.2 mm
- net Net-(S1-Pad2): track 6.53 -> 0.00 mm
- net /PowerTimer/EN_OUT: track 0.00 -> 5.61 mm
- net Net-(JP42-A): track 5.40 -> 0.00 mm
- net /PowerTimer/LOGIC_OUT: track 0.00 -> 4.48 mm
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- added copper zone on F.Cu, net BATT_IN
- added copper zone on In1.Cu, net BATT_IN
- added copper zone on In2.Cu, net GND
- added copper zone on In1.Cu, net VBUS
- added copper zone on In1.Cu, net VCC
Other:
- outline, holes or cut-outs redrawn
- copper layers 2 -> 4
- board text added: "9/24/23"
- board text removed: "9/4/23"

Commit message: Shit! Chinese new year
Parts:
- added C2: 0.1uF, Capacitor_SMD:C_0805_2012Metric_Pad1.18x1.45mm_HandSolder, F.Cu at (149.6, 105.0)
- added R2: 10k, Resistor_SMD:R_0805_2012Metric_Pad1.20x1.40mm_HandSolder, F.Cu at (148.5, 108.8)
- added U2: TMP117AIDRVT, TMP117AIDRVT:SON65P200X200X80-7N, F.Cu at (146.1, 105.9)
- J8: footprint Connector_JST:JST_XH_S4B-XH-A_1x04_P2.50mm_Horizontal -> Connector_PinHeader_2.54mm:PinHeader_1x04_P2.54mm_Vertical
- R1: value 10k -> 150
- moved J8 7.32 mm to (160.0, 75.4), turned to 90 degrees
- moved D1 3.56 mm to (138.3, 103.8)
- moved JP1 3.56 mm to (140.2, 107.8)
- moved D2 3.56 mm to (141.9, 103.8)
Connections:
- D3 pad 2: /PowerTimer/TEST_OUT -> /TEST
- J10 pad 13: unconnected-(J10-Pin_13) -> /TEST
- J8 pad 2: unconnected-(J8-Pin_2) -> GND
- J8 pad 3: unconnected-(J8-Pin_3) -> +5V
- SW1 pad 2: /PowerTimer/TEST_OUT -> /TEST
Routing:
- net /TEST: track 0.00 -> 80.8 mm, vias 0 -> 1
- net VBUS: track 47.5 -> 62.6 mm, vias 5 -> 6
- net /PowerTimer/LOGIC_OUT: track 4.48 -> 18.5 mm
- net +5V: track 25.4 -> 36.7 mm
- net /PowerTimer/TEST_OUT: track 9.48 -> 0.00 mm
- net /SDA: track 124.8 -> 132.6 mm, vias 2 -> 4
- net /SCL: track 122.9 -> 127.4 mm
- net Net-(BT2-+): track 47.7 -> 45.3 mm
- net Net-(U2-ADD0): track 0.00 -> 2.43 mm
- net GND: track 75.1 -> 77.5 mm, vias 28 -> 29
Other:
- board text added: "+5V"
- board text added: "3.3V"
- board text added: "BAT+"
- board text added: "HOLD"
- board text added: "SCL"
- board text added: "SDA"
