File: PowerMonitor.kicad_sch (KiCad schematic)
At the start: 6 parts

Commit message: Post-build updates
Parts:
- C: Mfr 1 (none) -> YAGEO; Mfr 1 PN (none) -> CC0805KRX7R9BB104; Supplier 1 Link (none) -> https://www.digikey.com/en/products/detail/yageo/CC0805KRX7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
- R: Mfr 1 (none) -> YAGEO; Mfr 1 PN (none) -> RC0805FR-0710RL; Supplier 1 Link (none) -> https://www.digikey.com/en/products/detail/yageo/RC0805FR-0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
- R: Mfr 1 (none) -> Stackpole Electronics Inc; Mfr 1 PN (none) -> RMCF2512FTR150; Supplier 1 Link (none) -> https://www.digikey.com/en/products/detail/stackpole-electr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
- U: Mfr 1 (none) -> Texas Instruments; Mfr 1 PN (none) -> INA219BIDR; Supplier 1 Link (none) -> https://www.digikey.com/en/products/detail/texas-instrument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
Changed lines of the file:
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@@
+      (effects (font (size 1.27 1.27)) hide)
+    )
+    (property "Mfr 1" "Texas Instruments" (id 4) (at 153.67 97.79 0)
+      (effects (font (size 1.27 1.27)) hide)
+    )
+    (property "Mfr 1 PN" "INA219BIDR" (id 5) (at 153.67 97.79 0)
+      (effects (font (size 1.27 1.27)) hide)
+    )
+    (property "Supplier 1 Link" "https://www.digikey.com/en/products/detail/texas-instruments/INA219BIDR/2426057" (id 6) (at 153.67 97.79 0)
       (effects (font (size 1.27 1.27)) hide)
     )
@@
       (effects (font (size 1.27 1.27)) hide)
     )
+    (property "Mfr 1" "YAGEO" (id 4) (at 128.27 97.79 0)
+      (effects (font (size 1.27 1.27)) hide)
+    )
+    (property "Mfr 1 PN" "CC0805KRX7R9BB104" (id 5) (at 128.27 97.79 0)
+      (effects (font (size 1.27 1.27)) hide)
+    )
+    (property "Supplier 1 Link" "https://www.digikey.com/en/products/detail/yageo/CC0805KRX7R9BB104/302874" (id 6) (at 128.27 97.79 0)
+      (effects (font (size 1.27 1.27)) hide)
+    )
     (pin "1")
     (pin "2")
@@
     )
     (property "Datasheet" "~" (id 3) (at 121.92 92.71 0)
+      (effects (font (size 1.27 1.27)) hide)
+    )
+    (property "Mfr 1" "YAGEO" (id 4) (at 121.92 92.71 0)
+      (effects (font (size 1.27 1.27)) hide)
+    )
+    (property "Mfr 1 PN" "RC0805FR-0710RL" (id 5) (at 121.92 92.71 0)
+      (effects (font (size 1.27 1.27)) hide)
+    )
+    (property "Supplier 1 Link" "https://www.digikey.com/en/products/detail/yageo/RC0805FR-0710RL/727534" (id 6) (at 121.92 92.71 0)
       (effects (font (size 1.27 1.27)) hide)
     )
@@
       (effects (font (size 1.27 1.27)) hide)
     )
+    (property "Mfr 1" "YAGEO" (id 4) (at 121.92 102.87 0)
+      (effects (font (size 1.27 1.27)) hide)
+    )
+    (property "Mfr 1 PN" "RC0805FR-0710RL" (id 5) (at 121.92 102.87 0)
+      (effects (font (size 1.27 1.27)) hide)
+    )
+    (property "Supplier 1 Link" "https://www.digikey.com/en/products/detail/yageo/RC0805FR-0710RL/727534" (id 6) (at 121.92 102.87 0)
+      (effects (font (size 1.27 1.27)) hide)
+    )
     (pin "1")
     (pin "2")
@@
     )
     (property "Datasheet" "~" (id 3) (at 111.76 97.79 0)
+      (effects (font (size 1.27 1.27)) hide)
+    )
+    (property "Mfr 1" "Stackpole Electronics Inc" (id 4) (at 111.76 97.79 0)
+      (effects (font (size 1.27 1.27)) hide)
+    )
+    (property "Mfr 1 PN" "RMCF2512FTR150" (id 5) (at 111.76 97.79 0)
+      (effects (font (size 1.27 1.27)) hide)
+    )
+    (property "Supplier 1 Link" "https://www.digikey.com/en/products/detail/stackpole-electronics-inc/RMCF2512FTR150/1716773?s=N4IgTCBcDaIBwFYAMBaASgWQMIDEwIEYwcAVNA5LElAOQBEQBdAXyA" (id 6) (at 111.76 97.79 0)
       (effects (font (size 1.27 1.27)) hide)
     )
@@
       (effects (font (size 1.27 1.27)) hide)
     )
+    (property "Mfr 1" "YAGEO" (id 4) (at 158.75 77.47 0)
+      (effects (font (size 1.27 1.27)) hide)
+    )
+    (property "Mfr 1 PN" "CC0805KRX7R9BB104" (id 5) (at 158.75 77.47 0)
+      (effects (font (size 1.27 1.27)) hide)
+    )
+    (property "Supplier 1 Link" "https://www.digikey.com/en/products/detail/yageo/CC0805KRX7R9BB104/302874" (id 6) (at 158.75 77.47 0)
+      (effects (font (size 1.27 1.27)) hide)
+    )
