File: PowerTimer.kicad_sch (KiCad schematic)
At the start: 20 parts

Commit message: technically ok
Parts:
- removed JP: SolderJumper_2_Bridged, symbol Jumper:SolderJumper_2_Bridged
- removed S: EG1213, EG1213:SW_EG1213, symbol EG1213:EG1213
- removed U: 74AUP1G32, symbol 74xGxx:74AUP1G32
- added D: LED, symbol Device:LED
- added R: R_Small, symbol Device:R_Small
- added SW: SW_Push_DPDT, symbol Switch:SW_Push_DPDT
- added U: 74AUC1G02, symbol 74xGxx:74AUC1G02
Connections:
- net GND: now also R.1, SW.3 (C), U.3 (GND)
- net INT: now also U.3 (~{INT}/SQW)
- net VCC: now also SW.6 (C), U.5 (VCC)
- net Vin: now also SW.1 (A)
- net at JP.2 (B): now also U.1
- net at JP.2 (B): now also U.2
- net EN_OUT: now reaches Q.1 (G)
- net EN_OUT: now also SW.5 (B)
- new net: D.1 (K), R.2
- new net LOGIC_OUT: SW.4 (A), U.4
- new net TEST_OUT: D.2 (A), SW.2 (B)
Other:
- note added: "NOR Gate 74AHC1G02"
- note removed: "OR Gate SN74AHC1G32"
- moved on the sheet: BT, C, D, J, Q, R, U
