File: PowerTimer.kicad_sch (KiCad schematic)
At the start: 21 parts

Commit message: Shit! Chinese new year
Parts:
- D: Mfr 1 (none) -> Everlight Elec; Mfr 1 PN (none) -> 17-21SURC/S530-A3/4T; Supplier 1 Link (none) -> C2943978
- J: Mfr 1 (none) -> NA; Mfr 1 PN (none) -> NA; Supplier 1 Link (none) -> NA
- Q: Mfr 1 (none) -> UMW(Youtai Semiconductor Co., Ltd.); Mfr 1 PN (none) -> IRLML2502; Supplier 1 Link (none) -> C347503
- R: Mfr 1 Stackpole Electronics Inc -> Viking Tech; Mfr 1 PN RNCP0805FTD10K0 -> AR05DTBW1500; Supplier 1 Link https://www.digikey.com/en/products/detail/stackpole-electr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 -> C2984396
- SW: Mfr 1 (none) -> C&K; Mfr 1 PN (none) -> JS202011SCQN; Supplier 1 Link (none) -> C221666
- U: Mfr 1 (none) -> Diodes Incorporated; Mfr 1 PN (none) -> 74AHC1G02W5-7; Supplier 1 Link (none) -> C842262
Changed lines of the file:
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@@
+      (effects (font (size 1.27 1.27)) hide)
+    )
+    (property "Mfr 1" "Diodes Incorporated" (id 4) (at 256.54 132.08 0)
+      (effects (font (size 1.27 1.27)) hide)
+    )
+    (property "Mfr 1 PN" "74AHC1G02W5-7" (id 5) (at 256.54 132.08 0)
+      (effects (font (size 1.27 1.27)) hide)
+    )
+    (property "Supplier 1 Link" "C842262" (id 6) (at 256.54 132.08 0)
       (effects (font (size 1.27 1.27)) hide)
     )
@@
       (effects (font (size 1.27 1.27)) hide)
     )
+    (property "Mfr 1" "NA" (id 4) (at 176.53 110.49 0)
+      (effects (font (size 1.27 1.27)) hide)
+    )
+    (property "Mfr 1 PN" "NA" (id 5) (at 176.53 110.49 0)
+      (effects (font (size 1.27 1.27)) hide)
+    )
+    (property "Supplier 1 Link" "NA" (id 6) (at 176.53 110.49 0)
+      (effects (font (size 1.27 1.27)) hide)
+    )
     (pin "1")
     (pin "2")
@@
     )
     (property "Datasheet" "~" (id 3) (at 304.8 179.07 0)
+      (effects (font (size 1.27 1.27)) hide)
+    )
+    (property "Mfr 1" "Everlight Elec " (id 4) (at 304.8 179.07 0)
+      (effects (font (size 1.27 1.27)) hide)
+    )
+    (property "Mfr 1 PN" "17-21SURC/S530-A3/4T" (id 5) (at 304.8 179.07 0)
+      (effects (font (size 1.27 1.27)) hide)
+    )
+    (property "Supplier 1 Link" "C2943978" (id 6) (at 304.8 179.07 0)
       (effects (font (size 1.27 1.27)) hide)
     )
@@
       (effects (font (size 1.27 1.27)) hide)
     )
-    (property "Mfr 1" "Stackpole Electronics Inc" (id 4) (at 304.8 190.5 0)
-      (effects (font (size 1.27 1.27)) hide)
-    )
-    (property "Mfr 1 PN" "RNCP0805FTD10K0" (id 5) (at 304.8 190.5 0)
-      (effects (font (size 1.27 1.27)) hide)
-    )
-    (property "Supplier 1 Link" "https://www.digikey.com/en/products/detail/stackpole-electronics-inc/RNCP0805FTD10K0/2240262" (id 6) (at 304.8 190.5 0)
+    (property "Mfr 1" "Viking Tech" (id 4) (at 304.8 190.5 0)
+      (effects (font (size 1.27 1.27)) hide)
+    )
+    (property "Mfr 1 PN" "AR05DTBW1500" (id 5) (at 304.8 190.5 0)
+      (effects (font (size 1.27 1.27)) hide)
+    )
+    (property "Supplier 1 Link" "C2984396" (id 6) (at 304.8 190.5 0)
       (effects (font (size 1.27 1.27)) hide)
     )
@@
     )
     (property "Datasheet" "~" (id 3) (at 293.37 139.7 0)
+      (effects (font (size 1.27 1.27)) hide)
+    )
+    (property "Mfr 1" "C&K" (id 4) (at 293.37 134.62 0)
+      (effects (font (size 1.27 1.27)) hide)
+    )
+    (property "Mfr 1 PN" "JS202011SCQN" (id 5) (at 293.37 134.62 0)
+      (effects (font (size 1.27 1.27)) hide)
+    )
+    (property "Supplier 1 Link" "C221666" (id 6) (at 293.37 134.62 0)
       (effects (font (size 1.27 1.27)) hide)
     )
@@
       (effects (font (size 1.27 1.27)) (justify left) hide)
     )
-    (pin "1")
+    (property "Mfr 1" "UMW(Youtai Semiconductor Co., Ltd.)" (id 4) (at 325.12 129.54 0)
+      (effects (font (size 1.27 1.27)) hide)
+    )
+    (property "Mfr 1 PN" "IRLML2502" (id 5) (at 325.12 129.54 0)
+      (effects (font (size 1.27 1.27)) hide)
+    )
+    (property "Supplier 1 Link" "C347503" (id 6) (at 325.12 129.54 0)
+      (effects (font (size 1.27 1.27)) hide)
+    )
+    (pin "1")
