File: PowerTimer.kicad_sch (KiCad schematic)
At the start: 19 parts

Commit message: PiShield!!
Parts:
- removed JP: SolderJumper_2_Bridged, symbol Jumper:SolderJumper_2_Bridged
- removed JP (x2): SolderJumper_3_Bridged12, symbol Jumper:SolderJumper_3_Bridged12
- removed JP: SolderJumper_3_Open, symbol Jumper:SolderJumper_3_Open
- removed U (x2): 74AUC2G02, symbol 74xGxx:74AUC2G02
- added JP (x3): SolderJumper_2_Open, symbol Jumper:SolderJumper_2_Open
- added R: R_Small, symbol Device:R_Small
- added S: EG1213, EG1213:SW_EG1213, symbol EG1213:EG1213
Connections:
- net ENABLE: now also S.2
- net GND: now also C.2; no longer C.1
- net NINT: now also JP.1 (A)
- net POWER_HOLD: now also JP.1 (A); no longer U.2
- net at U.1: now also JP.2 (B)
- net at U.4: now also JP.1 (A), R.1
- net +BATT renamed VCC
- net VCC: now also S.1; no longer C.2
- net VBUS renamed Vin
- new net: C.1, JP.2 (B), R.2, S.3
- new net: JP.2 (B), U.2
Other:
- note removed: "SR Latch 74LVC2G02"
- moved on the sheet: C, U

Commit message: Ready to order.
Parts:
- added D (x2): D_Schottky, symbol Device:D_Schottky
- added J: Conn_01x02_Male, symbol Connector:Conn_01x02_Male
- added JP: SolderJumper_2_Bridged, symbol Jumper:SolderJumper_2_Bridged
Connections:
- net GND: now also J.1 (Pin_1)
- net VCC: now also JP.2 (B); no longer BT.1 (+), U.14 (VBAT)
- net Vin: now also D.2 (A)
- new net: D.1 (K), D.1 (K), JP.1 (A)
- new net: BT.1 (+), D.2 (A), J.2 (Pin_2), U.14 (VBAT)
Other:
- note added: "Interrupt Inverter 74AHC1GU04"
- note added: "OR Gate SN74AHC1G32"
- note removed: "Interrupt Inverter 74LVC1GU04"
- note removed: "OR Gate 74LVC2G02"
- moved on the sheet: BT, JP

Commit message: Post-build updates
Parts:
- removed C: C_Small, symbol Device:C_Small
- removed JP: SolderJumper_2_Open, symbol Jumper:SolderJumper_2_Open
- removed R: R_Small, symbol Device:R_Small
- added Q: IRLML0030, Package_TO_SOT_SMD:SOT-23, symbol Transistor_FET:IRLML0030
- BT: Mfr 1 (none) -> Keystone Electronics; Mfr 1 PN (none) -> 3002TR; Supplier 1 Link (none) -> https://www.digikey.com/en/products/detail/keystone-electro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
- C: Mfr 1 (none) -> YAGEO; Mfr 1 PN (none) -> CC0805KRX7R9BB104; Supplier 1 Link (none) -> https://www.digikey.com/en/products/detail/yageo/CC0805KRX7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
- C: Mfr 1 (none) -> Samsung Electro-Mechanics; Mfr 1 PN (none) -> CL21A106KOCLRNC; Supplier 1 Link (none) -> https://www.digikey.com/en/products/detail/samsung-electro-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
- D: Mfr 1 (none) -> STMicroelectronics; Mfr 1 PN (none) -> BAT20JFILM; Supplier 1 Link (none) -> https://www.digikey.com/en/products/detail/stmicroelectroni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
- JP: Mfr 1 (none) -> NA; Mfr 1 PN (none) -> NA; Supplier 1 Link (none) -> NA
- R: Mfr 1 (none) -> Stackpole Electronics Inc; Mfr 1 PN (none) -> RNCP0805FTD10K0; Supplier 1 Link (none) -> https://www.digikey.com/en/products/detail/stackpole-electr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
- R: Mfr 1 (none) -> Stackpole Electronics Inc; Mfr 1 PN (none) -> RMCF0805JT470Kf; Supplier 1 Link (none) -> https://www.digikey.com/en/products/detail/stackpole-electr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
- S: Mfr 1 (none) -> E-Switch; Mfr 1 PN (none) -> EG1213; Supplier 1 Link (none) -> https://www.digikey.com/en/products/detail/e-switch/EG1213/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
- U: Mfr 1 (none) -> Analog Devices Inc./Maxim Integrated; Mfr 1 PN (none) -> DS3231M+; Supplier 1 Link (none) -> https://www.digikey.com/en/products/detail/analog-devices-i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
- U: Mfr 1 (none) -> Texas Instruments; Mfr 1 PN (none) -> SN74AHC1G32DBVR; Supplier 1 Link (none) -> https://www.digikey.com/en/products/detail/texas-instrument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
- U: Mfr 1 (none) -> Texas Instruments; Mfr 1 PN (none) -> SN74AHC1GU04DBVR; Supplier 1 Link (none) -> https://www.digikey.com/en/products/detail/texas-instrument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
Connections:
- net ENABLE: now also Q.3 (D); no longer S.2
- net GND: now also Q.2 (S)
- net at S.3: now also U.4
- new net: Q.1 (G), S.2
Other:
- moved on the sheet: BT, C, D, J, R, S, U

Commit message: revert to single layer
Parts:
- removed U: 74AUP1G32, symbol 74xGxx:74AUP1G32
- added U: 74AHC1G02, symbol 74xGxx:74AHC1G02
Connections:
- net GND: now also U.3 (GND)
- net VCC: now also U.5 (VCC)
- net at JP.2 (B): now also U.1
- net at JP.2 (B): now also U.2
- net at S.3: now also U.4
Changed lines of the file:
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@@
     (pin "9")
   )
-  (symbol (lib_id "74xGxx:74AUP1G32") (at 193.04 137.16 0) (unit 1)
-    (in_bom yes) (on_board yes)
-    (default_instance (reference "U") (unit 1) (value "74AUP1G32") (footprint ""))
-    (property "Reference" "U" (id 0) (at 180.34 129.54 0)
+  (symbol (lib_id "74xGxx:74AHC1G02") (at 193.04 137.16 0) (unit 1)
+    (in_bom yes) (on_board yes) (fields_autoplaced)
+    (default_instance (reference "U") (unit 1) (value "74AHC1G02") (footprint ""))
+    (property "Reference" "U" (id 0) (at 192.405 130.81 0)
       (effects (font (size 1.27 1.27)))
     )
-    (property "Value" "74AUP1G32" (id 1) (at 185.42 132.08 0)
+    (property "Value" "74AHC1G02" (id 1) (at 192.405 133.35 0)
       (effects (font (size 1.27 1.27)))
     )
@@
       (effects (font (size 1.27 1.27)) hide)
     )
-    (property "Mfr 1" "Texas Instruments" (id 4) (at 193.04 137.16 0)
-      (effects (font (size 1.27 1.27)) hide)
-    )
-    (property "Mfr 1 PN" "SN74AHC1G32DBVR" (id 5) (at 193.04 137.16 0)
-      (effects (font (size 1.27 1.27)) hide)
-    )
-    (property "Supplier 1 Link" "https://www.digikey.com/en/products/detail/texas-instruments/SN74AHC1G32DBVR/276737" (id 6) (at 193.04 137.16 0)
-      (effects (font (size 1.27 1.27)) hide)
-    )

Commit message: Update readme
Connections:
- net GND: now also S.1
- net VCC: no longer S.1
Other:
- moved on the sheet: BT, C, D, J, Q, R, S, U
