File: _autosave-BuoyPower.kicad_sch (KiCad schematic)
At the start: 13 parts

Commit message: Shit! Chinese new year
Parts:
- U: Mfr 1 (none) -> TMP117AIDRVT; Mfr 1 PN (none) -> Texas Instruments
Changed lines of the file:
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@@
       (effects (font (size 1.27 1.27)) (justify bottom) hide)
+    )
+    (property "Mfr 1" "TMP117AIDRVT" (id 17) (at 111.76 172.72 0)
+      (effects (font (size 1.27 1.27)) hide)
+    )
+    (property "Mfr 1 PN" "Texas Instruments" (id 18) (at 111.76 172.72 0)
+      (effects (font (size 1.27 1.27)) hide)
     )
     (pin "1")
@@
       (reference "#PWR0104") (unit 1) (value "VBUS") (footprint "")
     )
-    (path "/c400b7ca-4a96-4108-9b9c-a6711a29ec1d"
-      (reference "#PWR0105") (unit 1) (value "GND") (footprint "")
-    )
     (path "/de169543-5d83-41be-9f62-27d902158e7a"
       (reference "#PWR0105") (unit 1) (value "GND") (footprint "")
@@
       (reference "#PWR0119") (unit 1) (value "VBUS") (footprint "")
     )
-    (path "/1cb871b0-a81b-4f2c-aada-0e6748e94c8a"
-      (reference "#PWR0120") (unit 1) (value "VBUS") (footprint "")
-    )
-    (path "/461feab3-fdbc-4f9a-8b36-1ca162198b11"
-      (reference "#PWR0120") (unit 1) (value "VBUS") (footprint "")
-    )
     (path "/f81f13d3-aba1-4a34-8534-0b62464bd47f"
       (reference "#PWR0120") (unit 1) (value "VBUS") (footprint "")
@@
       (reference "#PWR0133") (unit 1) (value "+5V") (footprint "")
     )
+    (path "/c400b7ca-4a96-4108-9b9c-a6711a29ec1d"
+      (reference "#PWR0134") (unit 1) (value "GND") (footprint "")
+    )
+    (path "/1cb871b0-a81b-4f2c-aada-0e6748e94c8a"
+      (reference "#PWR0135") (unit 1) (value "VBUS") (footprint "")
+    )
+    (path "/461feab3-fdbc-4f9a-8b36-1ca162198b11"
+      (reference "#PWR0136") (unit 1) (value "VBUS") (footprint "")
+    )
     (path "/6d14d4f8-5eac-41fa-a6a0-78893e5397f9/c8ca51b5-6dd1-4daa-b0d5-f87bbc185ed8"
